File: VCA-2164.kicad_sch (KiCad schematic)
At the start: 108 parts, among them J1 AudioJack2_SwitchT, J10 AudioJack2_SwitchT, J11 AudioJack2_SwitchT, J12 AudioJack2_SwitchT, J13 AudioJack2, J14 Conn_02x05_Odd_Even, J15 Conn_01x01, J16 Conn_01x01, J17 Conn_01x01, J18 Conn_01x01, J19 Conn_01x01, J2 AudioJack2_SwitchT, J20 Conn_01x01, J21 Conn_01x01, J22 Conn_01x01, J23 Conn_01x01, J24 Conn_01x01, J25 Conn_01x01, J26 Conn_01x01, J27 Conn_01x01, J28 Conn_01x01, J29 Conn_01x01, J3 AudioJack2_SwitchT, J30 Conn_01x01, J31 Conn_01x01, J4 AudioJack2_SwitchT, J5 AudioJack2_SwitchT, J6 AudioJack2_SwitchT, J7 AudioJack2_SwitchT, J8 AudioJack2_SwitchT, J9 AudioJack2_SwitchT, U1 TL074, U2 AS2164, U3 TL074, U4 TL072

Commit message: non inverting outputs, peak indicator LED
Parts:
- added C10, C11, C12, C9: 100p, Capacitor_THT:C_Disc_D5.1mm_W3.2mm_P5.00mm, symbol Device:C
- added C27, C28: 0.1u, Capacitor_THT:C_Disc_D5.1mm_W3.2mm_P5.00mm, symbol Device:C
- added D1: 1N4148, Diode_THT:D_DO-35_SOD27_P7.62mm_Horizontal, symbol Diode:1N4148
- added D2: LED, Package_TO_SOT_THT:TO-92_Inline, symbol Device:LED
- added J32, J33, J34: Conn_01x01, Connector_Pin:Pin_D1.0mm_L10.0mm, symbol Connector_Generic:Conn_01x01
- added Q1, Q2: BC556, Package_TO_SOT_THT:TO-92_Wide, symbol Transistor_BJT:BC556
- added R25, R26, R27, R28, R29, R30, R31, R32, R45: 10k, Resistor_THT:R_Axial_DIN0207_L6.3mm_D2.5mm_P10.16mm_Horizontal, symbol Device:R
- added R46: 100k, Resistor_THT:R_Axial_DIN0207_L6.3mm_D2.5mm_P10.16mm_Horizontal, symbol Device:R
- added R47, R48, R49: 750, Resistor_THT:R_Axial_DIN0207_L6.3mm_D2.5mm_P10.16mm_Horizontal, symbol Device:R
- added U4: TL074, Package_DIP:DIP-14_W7.62mm_Socket, symbol Amplifier_Operational:TL074
- C13: renamed from C11; value 100p -> 22p
- C14: renamed from C9; value 100p -> 22p
- C15: renamed from C10; value 100p -> 22p
- C16: renamed from C12; value 100p -> 22p
- C17: renamed from C13; value 100p -> 22p
- C18: renamed from C14; value 100p -> 22p
- U3: footprint Package_DIP:DIP-14_W7.62mm_Socket -> (none)
- renumbered C15 to C19, C16 to C20, C17 to C21, C18 to C22, C19 to C23, C20 to C24, C21 to C25, C22 to C26, C23 to C29, C24 to C30, J9 to J10, J10 to J11, J11 to J9, R23 to R21, R21 to R23, R26 to R33, R25 to R34, R28 to R35, R27 to R36, R29 to R37, R30 to R38, R31 to R39, R32 to R40, R33 to R41, R34 to R42, R35 to R43, R36 to R44, R37 to R50, U4 to U5
Connections:
- net GND: now also U3.10 (+), U3.12 (+), C27.2, C28.1, D2.1 (K), J33.1 (Pin_1), R46.1, R47.1, U4.10 (+), U4.12 (+), U4.3 (+), U4.5 (+); no longer U3.10 (+), U3.12 (+)
- net VCC: now also C27.1, J32.1 (Pin_1), R48.2, U4.4 (V+)
- net VEE: now also C28.2, U4.11 (V-)
- net at R24.1, U2.13: now also C12.1, U4.6 (-); no longer C16.1, U3.2 (-)
- net at C16.2, R36.1: now also R32.2, U4.1; no longer R24.2, U3.1
- net at C15.2, R34.1: now also U3.14, R30.2; no longer R22.2, U3.8
- net at R22.1, U2.5: now also U3.9 (-), C10.1; no longer C15.1, U3.9 (-)
- net at R21.1, U2.12, U3.6 (-): now also C9.1; no longer C13.1
- net at C13.2, R33.1: now also U3.1, R29.2; no longer R21.2, U3.7
- net at R23.1, U2.4: now also C11.1, U4.9 (-); no longer C14.1, U3.13 (-)
- net at C14.2, R35.1: now also R31.2, U4.14; no longer R23.2, U3.14
- net at C18.2, R43.2, R44.1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: now also D1.2 (A)
- new net: C12.2, R24.2, R28.1, U4.7
- new net: C16.1, R28.2, R32.1, U4.2 (-)
- new net: C15.1, R26.2, R30.1, U3.13 (-)
- new net: C13.1, R25.2, R29.1, U3.2 (-)
- new net: C9.2, R21.2, R25.1, U3.7
- new net: D1.1 (K), R45.1
- new net: Q1.2 (B), R45.2, R46.2
- new net: C10.2, R22.2, R26.1, U3.8
- new net: C11.2, R23.2, R27.1, U4.8
- new net: Q1.3 (E), Q2.3 (E), R48.1
- new net: C14.1, R27.2, R31.1, U4.13 (-)
- new net: Q1.1 (C), Q2.2 (B), R47.2
- new net: Q2.1 (C), R49.2
- new net LED_A: D2.2 (A), J34.1 (Pin_1), R49.1
Other:
- moved on the sheet: C1, C13, C14, C15, C16, C17, C18, C2, C29, C3, C30, C4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

Commit message: unnecessary cap
Parts:
- removed C17: 22p, Capacitor_THT:C_Disc_D5.1mm_W3.2mm_P5.00mm, symbol Device:C
- renumbered C18 to C17, C19 to C18, C20 to C19, C21 to C20, C22 to C21, C23 to C22, C24 to C23, C25 to C24, C26 to C25, C27 to C26, C28 to C27, C29 to C28, C30 to C29
Changed lines of the file:
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@@
 	)
 	(junction
-		(at 337.82 129.54)
-		(diameter 0)
-		(color 0 0 0 0)
-	)
-	(junction
 		(at 236.22 287.02)
 		(diameter 0)
@@
 	(wire
 		(pts
-			(xy 314.96 129.54) (xy 322.58 129.54)
-		)
-		(stroke
-			(width 0)
-			(type default)
-		)
-	)
-	(wire
-		(pts
 			(xy 222.25 373.38) (xy 228.6 373.38)
 		)
@@
 	(wire
 		(pts
-			(xy 330.2 129.54) (xy 337.82 129.54)
-		)
-		(stroke
-			(width 0)
-			(type default)
-		)
-	)
-	(wire
-		(pts
 			(xy 449.58 196.85) (xy 420.37 196.85)
 		)
@@
 		(dnp no)
 		(fields_autoplaced yes)
-		(property "Reference" "C24"
+		(property "Reference" "C23"
 			(at 457.2 72.3899 0)
 			(show_name no)
@@
 			(project "VCA-2164"
 				(path "/682d00d9-e143-43dd-923f-005dee495aa3"
-					(reference "C24")
+					(reference "C23")
 					(unit 1)
 				)
@@
 		(dnp no)
 		(fields_autoplaced yes)
-		(property "Reference" "C27"
+		(property "Reference" "C26"
 			(at 478.79 58.4199 0)
 			(show_name no)
@@
 			(project "VCA-2164"
 				(path "/682d00d9-e143-43dd-923f-005dee495aa3"
-					(reference "C27")
+					(reference "C26")
 					(unit 1)
 				)
@@
 	(symbol
 		(lib_id "Device:C")
-		(at 326.39 129.54 90)
-		(unit 1)
-		(body_style 1)
-		(exclude_from_sim no)
-		(in_bom yes)
-		(on_board yes)
-		(in_pos_files yes)
-		(dnp no)
-		(fields_autoplaced yes)
-		(property "Reference" "C17"
-			(at 326.39 121.92 90)
-			(show_name no)
-			(do_not_autoplace no)
-			(effects
-				(font
-					(size 1.27 1.27)
-				)
-			)
-		)
-		(property "Value" "22p"
-			(at 326.39 124.46 90)
-			(show_name no)
-			(do_not_autoplace no)
-			(effects
-				(font
-					(size 1.27 1.27)
-				)
-			)
-		)
-		(property "Footprint" "Capacitor_THT:C_Disc_D5.1mm_W3.2mm_P5.00mm"
-			(at 330.2 128.5748 0)
-			(hide yes)
-			(show_name no)
-			(do_not_autoplace no)
-			(effects
-				(font
-					(size 1.27 1.27)
-				)
-			)
-		)
-		(property "Datasheet" ""
-			(at 326.39 129.54 0)
-			(hide yes)
-			(show_name no)
-			(do_not_autoplace no)
-			(effects
-				(font
-					(size 1.27 1.27)
-				)
-			)
-		)
-		(property "Description" "Unpolarized capacitor"
-			(at 326.39 129.54 0)
-			(hide yes)
-			(show_name no)
-			(do_not_autoplace no)
-			(effects
-				(font
-					(size 1.27 1.27)
-				)
-			)
-		)
-		(pin "1"
-		)
-		(pin "2"
-		)
-		(instances
-			(project "VCA-2164"
-				(path "/682d00d9-e143-43dd-923f-005dee495aa3"
-					(reference "C17")
-					(unit 1)
-				)
-			)
-		)
-	)
-	(symbol
-		(lib_id "Device:C")
 		(at 147.32 119.38 0)
 		(unit 1)
@@
 		(dnp no)
 		(fields_autoplaced yes)
-		(property "Reference" "C21"
+		(property "Reference" "C20"
 			(at 445.77 58.4199 0)
 			(show_name no)
@@
 			(project "VCA-2164"
 				(path "/682d00d9-e143-43dd-923f-005dee495aa3"
-					(reference "C21")
+					(reference "C20")
 					(unit 1)
 				)
@@
 		(dnp no)
 		(fields_autoplaced yes)
-		(property "Reference" "C29"
+		(property "Reference" "C28"
 			(at 534.67 195.5799 0)
 			(show_name no)
@@
 			(project "VCA-2164"
 				(path "/682d00d9-e143-43dd-923f-005dee495aa3"
-					(reference "C29")
+					(reference "C28")
 					(unit 1)
 				)
@@
 		(dnp no)
 		(fields_autoplaced yes)
-		(property "Reference" "C23"
+		(property "Reference" "C22"
 			(at 457.2 58.4199 0)
 			(show_name no)
@@
 			(project "VCA-2164"
 				(path "/682d00d9-e143-43dd-923f-005dee495aa3"
-					(reference "C23")
+					(reference "C22")
 					(unit 1)
 				)
@@
 		(dnp no)
 		(fields_autoplaced yes)
-		(property "Reference" "C30"
+		(property "Reference" "C29"
 			(at 539.75 166.3699 0)
 			(show_name no)
@@
 			(project "VCA-2164"
 				(path "/682d00d9-e143-43dd-923f-005dee495aa3"
-					(reference "C30")
+					(reference "C29")
 					(unit 1)
 				)
@@
 		(dnp no)
 		(fields_autoplaced yes)
-		(property "Reference" "C26"
+		(property "Reference" "C25"
 			(at 467.36 72.3899 0)
 			(show_name no)
@@
 			(project "VCA-2164"
 				(path "/682d00d9-e143-43dd-923f-005dee495aa3"
-					(reference "C26")
+					(reference "C25")
 					(unit 1)
 				)
@@
 		(dnp no)
 		(fields_autoplaced yes)
-		(property "Reference" "C25"
+		(property "Reference" "C24"
 			(at 467.36 58.4199 0)
 			(show_name no)
@@
 			(project "VCA-2164"
 				(path "/682d00d9-e143-43dd-923f-005dee495aa3"
-					(reference "C25")
+					(reference "C24")
 					(unit 1)
 				)
@@
 		(dnp no)
 		(fields_autoplaced yes)
-		(property "Reference" "C19"
+		(property "Reference" "C18"
 			(at 422.91 57.5309 0)
 			(show_name no)
@@
 			(project "VCA-2164"
 				(path "/682d00d9-e143-43dd-923f-005dee495aa3"
-					(reference "C19")
+					(reference "C18")
 					(unit 1)
 				)
@@
 		(dnp no)
 		(fields_autoplaced yes)
-		(property "Reference" "C28"
+		(property "Reference" "C27"
 			(at 478.79 72.3899 0)
 			(show_name no)
@@
 			(project "VCA-2164"
 				(path "/682d00d9-e143-43dd-923f-005dee495aa3"
-					(reference "C28")
+					(reference "C27")
 					(unit 1)
 				)
@@
 		(dnp no)
 		(fields_autoplaced yes)
-		(property "Reference" "C18"
+		(property "Reference" "C17"
 			(at 368.3 121.92 90)
 			(show_name no)
@@
 			(project "VCA-2164"
 				(path "/682d00d9-e143-43dd-923f-005dee495aa3"
-					(reference "C18")
+					(reference "C17")
 					(unit 1)
 				)
@@
 		(dnp no)
 		(fields_autoplaced yes)
-		(property "Reference" "C22"
+		(property "Reference" "C21"
 			(at 445.77 72.3899 0)
 			(show_name no)
@@
 			(project "VCA-2164"
 				(path "/682d00d9-e143-43dd-923f-005dee495aa3"
-					(reference "C22")
+					(reference "C21")
 					(unit 1)
 				)
@@
 		(dnp no)
 		(fields_autoplaced yes)
-		(property "Reference" "C20"
+		(property "Reference" "C19"
 			(at 422.91 71.5009 0)
 			(show_name no)
@@
 			(project "VCA-2164"
 				(path "/682d00d9-e143-43dd-923f-005dee495aa3"
-					(reference "C20")
+					(reference "C19")
 					(unit 1)
 				)
